Commit message: guardar todo

File: delta_description/diffdrive_urdf/lidar.xacro (robot description, xacro)
@@ -30,4 +30,5 @@
         <topic>scan</topic>
         <gz_frame_id>lidar_link</gz_frame_id>
+        <pose relative_to='lidar_link'>0 0 0 0 0 0</pose>
         <lidar>
         <scan>

File: delta_description/diffdrive_urdf/robot.urdf.xacro (robot description, xacro)
@@ -1,11 +1,23 @@
 <?xml version="1.0"?>
 <robot xmlns:xacro="http://www.ros.org/wiki/xacro" name="delta_robot">
+    <!-- Example link -->
     <xacro:include filename="properties.xacro"/>
     <xacro:include filename="robot_core.xacro"/>
-    <!-- LIDAR -->
+    <!-- Lidar sensor -->
     <xacro:include filename="lidar.xacro"/>
+    <!-- IMU sensor -->
+    <xacro:include filename="imu_sensor.xacro"/>
+    <!-- Depth camera sensor -->
+    <xacro:include filename="camera.xacro"/>
     <!-- ros2_control -->
     <xacro:include filename="ros2_control.xacro"/>
-    <xacro:include filename="imu_sensor.xacro"/>
-    <xacro:include filename="camera.xacro"/>
+    <!-- <gazebo>
+      <plugin filename="libgz-sim-pose-publisher-system.so" name="gz::sim::systems::PosePublisher">
+        <publish_link_pose>false</publish_link_pose>
+        <publish_model_pose>true</publish_model_pose>
+        <publish_nested_model_pose>true</publish_nested_model_pose>
+        <use_pose_vector_msg>false</use_pose_vector_msg>
+        <update_frequency>50</update_frequency>
+      </plugin>
+    </gazebo> -->
 </robot>

File: delta_description/diffdrive_urdf/robot_core.xacro (robot description, xacro)
@@ -53,18 +53,16 @@
         <collision>
             <geometry>
-                <sphere radius="${rad_w}" />
+                  <sphere radius="${rad_w}" />
             </geometry>
-        <surface>
-            <friction>
-                <ode>
-                <mu1>2</mu1>
-                <mu2>4</mu2>
-                <kp>1000000.0</kp>
-                <kd>10.0</kd>
-                </ode>
-            </friction>
-        </surface>
+            <surface>
+                <friction>
+                    <ode>
+                        <mu>1.0</mu>
+                        <mu2>2.0</mu2>
+                    </ode>
+                </friction>
+            </surface>
         </collision>
-        <xacro:inertial_cylinder mass="0.5" length="${le_w}" radius="${rad_w}">
+        <xacro:inertial_cylinder mass="0.1" length="${le_w}" radius="${rad_w}">
             <origin xyz="0 0 0" rpy="0 0 0"/>
         </xacro:inertial_cylinder>
@@ -88,18 +86,16 @@
         <collision>
             <geometry>
-                <sphere radius="${rad_w}" />
+                  <sphere radius="${rad_w}" />
             </geometry>
             <surface>
                 <friction>
-                <ode>
-                <mu1>2</mu1>
-                <mu2>4</mu2>
-                <kp>1000000.0</kp>
-                <kd>10.0</kd>
-                </ode>
+                    <ode>
+                        <mu>1.0</mu>
+                        <mu2>2.0</mu2>
+                    </ode>
                 </friction>
             </surface>
         </collision>
-        <xacro:inertial_cylinder mass="0.5" length="${le_w}" radius="${rad_w}">
+        <xacro:inertial_cylinder mass="0.1" length="${le_w}" radius="${rad_w}">
             <origin xyz="0 0 0" rpy="0 0 0"/>
         </xacro:inertial_cylinder>
